File: ploter_cnc.kicad_sch (KiCad schematic)
At the start: 9 parts, among them J1 Conn_01x05_Socket, J2 Conn_01x05_Socket, J3 Conn_01x05_Socket, J4 Conn_01x02_Socket, U1 ULN2803A, U2 ULN2803A

Commit message: primera version a imprimir
Parts:
- removed C2: 100mf, symbol Device:C
- added C2: 100 µF, Capacitor_THT:CP_Radial_D4.0mm_P2.00mm, symbol Device:C_Polarized
- added H1, H2, H3, H4: MountingHole, MountingHole:MountingHole_2.2mm_M2_DIN965_Pad, symbol Mechanical:MountingHole
- C1: value 100nf -> 100 nf; footprint (none) -> Capacitor_THT:C_Disc_D4.3mm_W1.9mm_P5.00mm
Connections:
- net GND: now also C2.2
- net VCC: now also C2.1

Commit message: xlas
Connections:
- net A: now also U1.18 (O1); no longer U1.1 (I1)
- net A1: now also J2.5 (Pin_5), U2.11 (O8); no longer J2.2 (Pin_2), U2.1 (I1)
- net A2: now also J3.5 (Pin_5), U2.15 (O4); no longer J3.2 (Pin_2), U2.5 (I5)
- net B: now also U1.17 (O2); no longer U1.2 (I2)
- net B1: now also J2.4 (Pin_4), U2.12 (O7); no longer J2.3 (Pin_3), U2.2 (I2)
- net B2: now also J3.4 (Pin_4), U2.16 (O3); no longer J3.3 (Pin_3), U2.6 (I6)
- net C: now also U1.16 (O3); no longer U1.3 (I3)
- net C1: now also J2.3 (Pin_3), U2.13 (O6); no longer J2.4 (Pin_4), U2.3 (I3)
- net C2: now also J3.3 (Pin_3), U2.17 (O2); no longer J3.4 (Pin_4), U2.7 (I7)
- net D: now also U1.15 (O4); no longer U1.4 (I4)
- net D1: now also J2.2 (Pin_2), U2.14 (O5); no longer J2.5 (Pin_5), U2.4 (I4)
- net D2: now also J3.2 (Pin_2), U2.18 (O1); no longer J3.5 (Pin_5), U2.8 (I8)
- net at U3.21 (GPIO16): now also U2.7 (I7); no longer U2.17 (O2)
- net at U3.22 (GPIO17): now also U2.6 (I6); no longer U2.16 (O3)
- net at U3.24 (GPIO18): now also U2.5 (I5); no longer U2.15 (O4)
- net at U3.25 (GPIO19): now also U2.4 (I4); no longer U2.14 (O5)
- net at U3.26 (GPIO21): now also U2.3 (I3); no longer U2.13 (O6)
- net at U3.29 (GPIO22): now also U2.2 (I2); no longer U2.12 (O7)
- net at U3.3 (GPIO13): now also U2.8 (I8); no longer U2.18 (O1)
- net at U3.30 (GPIO23): now also U2.1 (I1); no longer U2.11 (O8)
- net at U3.5 (GPIO14): now also U1.1 (I1); no longer U1.15 (O4)
- net at U3.6 (GPIO27): now also U1.2 (I2); no longer U1.16 (O3)
- net at U3.7 (GPIO26): now also U1.3 (I3); no longer U1.17 (O2)
- net at U3.8 (GPIO25): now also U1.4 (I4); no longer U1.18 (O1)
Other:
- note added: "//3 grupos 25,26,27,14 13,16,17,18 19,21,22,23"
- moved on the sheet: J1, J2, J3, U1, U2
